Commit message: gazeboSim done

File: urdf/my_robot.urdf.xacro (robot description, xacro)
@@ -1,4 +1,5 @@
 <?xml version="1.0"?>
 <robot xmlns:xacro="http://www.ros.org/wiki/xacro" name="my_robot">
+    <xacro:include filename="gazebo_control.xacro" />
     <material name="white">
         <color rgba="1 1 1 1" />
@@ -28,5 +29,6 @@
     <!-- Caster wheel position - at the back -->
     <xacro:property name="caster_x_offset" value="-0.05" /> <!-- -base_length/2 = -78mm -->
-    <xacro:property name="caster_z_offset" value="-0.034" /> <!-- below base -->
+    <xacro:property name="fcaster_x_offset" value="0.05" /> <!-- -base_length/2 = -78mm -->
+    <xacro:property name="caster_z_offset" value="-0.030" /> <!-- below base -->
     <!-- ========== CYLINDER MACRO ========== -->
     <xacro:macro name="vertical_cylinder" params="name x y z color">
@@ -73,4 +75,7 @@
         </inertial>
     </link>
+    <gazebo reference="base_link">
+        <material>Gazebo/Black</material>
+    </gazebo>
     <!-- ========== TOP PLATE ========== -->
     <link name="top_plate">
@@ -97,4 +102,7 @@
     <origin xyz="0 0 0.060" rpy="0 0 0"/>
     </joint>
+    <gazebo reference="top_plate">
+        <material>Gazebo/Grey</material>
+    </gazebo>
     <!-- Front Left -->
     <xacro:vertical_cylinder name="front_left_cylinder" x="0.065" y="0.062" z="0.040" color="silver"/>
@@ -105,4 +113,16 @@
     <!-- Rear Right -->
     <xacro:vertical_cylinder name="rear_right_cylinder" x="-0.065" y="-0.062" z="0.040" color="silver"/>
+    <gazebo reference="front_left_cylinder">
+        <material>Gazebo/Silver</material>
+    </gazebo>
+    <gazebo reference="front_right_cylinder">
+        <material>Gazebo/Silver</material>
+    </gazebo>
+    <gazebo reference="rear_left_cylinder">
+        <material>Gazebo/Silver</material>
+    </gazebo>
+    <gazebo reference="rear_left_cylinder">
+        <material>Gazebo/Silver</material>
+    </gazebo>
     <!-- ========== FRONT BLOCK ========== -->
     <link name="front_block">
@@ -129,4 +149,7 @@
     <origin xyz="0.057 0.0 0" rpy="0 0 0"/>
     </joint>
+    <gazebo reference="front_block">
+        <material>Gazebo/Black</material>
+    </gazebo>
      <!-- ========== REAR BLOCK ========== -->
     <link name="rear_block">
@@ -153,4 +176,7 @@
     <origin xyz="-0.057 0.0 0" rpy="0 0 0"/>
     </joint>
+    <gazebo reference="rear_block">
+        <material>Gazebo/Black</material>
+    </gazebo>
     <!-- ========== LEFT WHEEL ========== -->
     <link name="left_wheel">
@@ -178,4 +204,7 @@
         <axis xyz="0 0 1"/>
     </joint>
+    <gazebo reference="left_wheel">
+        <material>Gazebo/Blue</material>
+    </gazebo>
     <!-- ========== RIGHT WHEEL ========== -->
     <link name="right_wheel">
@@ -203,4 +232,7 @@
         <axis xyz="0 0 -1"/>
     </joint>
+    <gazebo reference="right_wheel">
+        <material>Gazebo/Blue</material>
+    </gazebo>
     <!-- ========== CASTER WHEEL ========== -->
     <link name="caster_wheel">
@@ -209,7 +241,5 @@
             <sphere radius="0.015"/>  <!-- 15mm radius -->
         </geometry>
-        <material name="gray">
-            <color rgba="0.5 0.5 0.5 1"/>
-        </material>
+        <material name="grey"/>
         </visual>
         <collision>
@@ -224,8 +254,11 @@
         </inertial>
     </link>
-    <joint name="caster_joint" type="fixed">
+    <joint name="caster_wheel_joint" type="fixed">
         <parent link="base_link"/>
         <child link="caster_wheel"/>
         <origin xyz="${caster_x_offset} 0 ${caster_z_offset}" rpy="0 0 0"/>
     </joint>
+    <gazebo reference="caster_wheel">
+        <material>Gazebo/Silver</material>
+    </gazebo>
 </robot>
